File: Z570M_socket/Z570M_socket.kicad_sch (KiCad schematic)
At the start: 3 parts, among them J1 Conn_01x06_Pin, J3 Conn_01x05_Pin

Commit message: edit Readme.md
Other:
- note removed: "When soldering, cool pins near the place where they enter the tube. Too much heat can cause vacuum leak. Red tube coating dissolves in water!"
- company: Tomas Kouba -> TK
- moved on the sheet: J1, J3, U1
